File: ADAU1787-eval.kicad_sch (KiCad schematic)
At the start: 1 part, among them U1 ADAU1787BCBZRL

Commit message: stuff
Parts:
- added C? (x3): 10u, symbol Device:C
- added C? (x6): 100n, symbol Device:C
- added C? (x2): C, symbol Device:C
- added C?: 1u, symbol Device:C
- added J?: AudioJack2, symbol Connector:AudioJack2
- added J?: Conn_Coaxial, symbol Connector:Conn_Coaxial
- added JP?: Jumper_3_Bridged12, symbol Jumper:Jumper_3_Bridged12
- added R?: 49.9, symbol Device:R
- added TP? (x12): TestPoint, symbol Connector:TestPoint
Connections:
- net DVDD: now reaches U1.A3 (DVDD)
- net DVDD: now also C?.1, C?.1, TP?.1
- net IOVDD: now reaches U1.A5 (IOVDD)
- net IOVDD: now also C?.1, C?.1, TP?.1
- net AVDD: now reaches U1.D1 (HPVDD)
- net AVDD: now also U1.E7 (AVDD), U1.F2 (AVDD), C?.1, C?.1, C?.1, C?.1, TP?.1, TP?.1, TP?.1
- net OUTPUT1_P: now reaches U1.E2 (HPOUTP0/LOUTP0)
- net OUTPUT1_P: now also TP?.1
- net INPUT4: now reaches U1.E4 (AIN3)
- net INPUT4: now also TP?.1
- net INPUT2: now reaches U1.E5 (AIN1)
- net INPUT2: now also TP?.1
- net OUTPUT1_N: now reaches U1.F1 (HPOUTN0/LOUTP0)
- net OUTPUT1_N: now also TP?.1
- net GND: now reaches U1.F3 (AGND)
- net GND: now also U1.F7 (AGND), C?.2, C?.2, C?.2, C?.2, C?.2, C?.2, C?.2, C?.2, C?.2, C?.2, C?.2, J?.2 (Ext), J?.S, R?.2
- net CM: now reaches U1.F4 (CM)
- net CM: now also C?.1, C?.1, TP?.1
- net INPUT3: now reaches U1.F5 (AIN2)
- net INPUT3: now also TP?.1
- net INPUT1: now reaches U1.F6 (AIN0)
- net INPUT1: now also C?.2, TP?.1
- new net: J?.T, JP?.1 (A)
- new net: C?.1, C?.1, JP?.2 (C), R?.1
- new net: J?.1 (In), JP?.3 (B)
Other:
- moved on the sheet: U1
